File: examples/TripleRecursion/FolderStructure.kicad_pcb (KiCad board)
At the start: 2 copper layers, 79.4 x 40.8 mm, 22 parts, among them J1 Screw_Terminal_01x04, J2 Screw_Terminal_01x04, J3 Screw_Terminal_01x04, Q1 MMBT2222A, Q2 BC807, Q3 MMBT2222A, Q4 BC807, Q5 MMBT2222A, Q6 BC807, U1 ATtiny1626-X

Commit message: Add Zones to Examples
Routing:
- added copper zone on F.Cu, net /SubPcb/Input
- added copper zone on F.Cu, net /SubPcb/nType/Output
- added copper zone on F.Cu, net /SubPcb1/Input
- added copper zone on F.Cu, net /SubPcb1/nType/Output
- added copper zone on F.Cu, net /SubPcb2/Input
- added copper zone on F.Cu, net /SubPcb2/nType/Output
- added copper zone on F.Cu, net GND
